File: IO4-SignalDriver.sch (EAGLE design)
At the start: 20 parts, among them CON1 CONNECTOR-RJ45-FRONT, IC1 74LS139N, P1 500R, P2 500R, P3 500R, P4 500R, P5 500R, P6 500R

Commit message: convert to SMT, add 2mmx4 headers
Parts:
- added CON2, CON3: CONNECTOR-GROVE-4P-2.0-3470130P1, SPCoast:CONNECTOR-GROVE-4P-2.0-3470130P1
- added FID1, FID2: FIDUCIAL, SPCoast:FIDUCIAL
- BOARD1: value (none) -> BOARD80X100
- C1: device rcl:C-US025-030X050 -> SPCoast:CAP0603
- CON1: value CONNECTOR-RJ45-FRONT -> (none)
- IC1: value 74LS139N -> 74LS139D; device 74xx-us:74LS139N -> SPCoast:74LS139D
- J1: device MCP:520250-3 -> SPCoast:CONNECTOR-RJ25-6P6C
- R1, R2, R3, R4, R5, R6: value 150R -> 470R; device SparkFun:RESISTORPTH-1/4W -> SPCoast:R0805-RES
Connections:
- net G1-LED: now also CON2.1
- net G2-LED: now also CON3.1
- net R1-LED: now also CON2.3
- net R2-LED: now also CON3.3
- net VCC: now also CON2.4, CON3.4
- net Y1-LED: now also CON2.2
- net Y2-LED: now also CON3.2
Other:
- note added: "2x 2mm 4-pin JST"
- note added: "CMRI Breakout"
- note added: "RJ45"
- note added: "RJ45 adapter"
- note added: "v3.1"

Commit message: changed silkscreen version info
Other:
- note added: "2.0"
- note removed: "1.8"
Changed lines of the file:
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@@
 <text x="149.098" y="26.924" size="5.08" layer="91">SPCoast</text>
 <text x="149.098" y="6.858" size="2.54" layer="91">Signal Control Circuit</text>
-<text x="237.236" y="5.842" size="5.08" layer="91">1.8</text>
+<text x="237.236" y="5.842" size="5.08" layer="91">2.0</text>
 <text x="60.96" y="53.34" size="3.81" layer="91" rot="R90">5V</text>
 <text x="72.644" y="14.224" size="2.54" layer="104">0b00 = GREEN

Commit message: removed unused sch sheet
Other:
- note removed: "CMRI Breakout"
- note removed: "RJ45 adapter"
- note removed: "v3.1"
Changed lines of the file:
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@@
 <part name="P+6" library="SparkFun" deviceset="VCC" device=""/>
 <part name="P+7" library="SparkFun" deviceset="VCC" device=""/>
-<part name="FRAME2" library="SparkFun" deviceset="FRAME-LETTER" device=""/>
 <part name="CON2" library="SPCoast" deviceset="CONNECTOR-GROVE-4P-2.0" device="-3470130P1"/>
 <part name="CON3" library="SPCoast" deviceset="CONNECTOR-GROVE-4P-2.0" device="-3470130P1"/>
@@
 </nets>
 </sheet>
-<sheet>
-<plain>
-<text x="152.4" y="27.94" size="3.81" layer="104">CMRI Breakout</text>
-<text x="198.12" y="27.94" size="3.81" layer="104">RJ45 adapter</text>
-<text x="236.22" y="7.62" size="3.81" layer="104">v3.1</text>
-</plain>
-<instances>
-<instance part="FRAME2" gate="G$1" x="0" y="0"/>
-<instance part="FRAME2" gate="G$2" x="147.32" y="0"/>
-</instances>
-<busses>
-</busses>
-<nets>
-</nets>
-</sheet>

Commit message: font=vector
Parts:
- R1, R2, R3, R4, R5, R6: value 470R -> 330R
- renumbered J2 to CON4, J3 to CON5
Other:
- note added: "(with individual brightness adjustments for each LED)"
- note added: "3.5mm Screw Term"
- note added: "IO4 Signal Driver"
- note added: "John Plocher"
- note removed: "SPCoast"
- note removed: "Signal Control Circuit"
- moved on the sheet: CON1, CON2, CON3
